Commit message: added rotation yaw 270 roll 270 to standard vtol and iris

File: models/rotors_description/urdf/iris_base.xacro (robot description, xacro)
@@ -82,5 +82,5 @@
   >
     <inertia ixx="0.00001" ixy="0.0" ixz="0.0" iyy="0.00001" iyz="0.0" izz="0.00001" />
-    <origin xyz="0 0 0" rpy="0 0 0" />
+    <origin xyz="0 0 0" rpy="-1.57 0 1.57" />
   </xacro:imu_plugin_macro>
   <xacro:if value="$(arg enable_ground_truth)">
@@ -102,5 +102,5 @@
     >
       <inertia ixx="0.00001" ixy="0.0" ixz="0.0" iyy="0.00001" iyz="0.0" izz="0.00001" />
-      <origin xyz="0 0 0" rpy="0 0 0" />
+      <origin xyz="0 0 0" rpy="-1.57 0 1.57" />
     </xacro:imu_plugin_macro>
     <!-- Mount a generic odometry sensor providing ground truth. -->

Commit message: made yaw 270 roll 90 rotation for standard_vtol and iris models

File: models/rotors_description/urdf/iris_base.xacro (robot description, xacro)
@@ -82,5 +82,5 @@
   >
     <inertia ixx="0.00001" ixy="0.0" ixz="0.0" iyy="0.00001" iyz="0.0" izz="0.00001" />
-    <origin xyz="0 0 0" rpy="-1.57 0 1.57" />
+    <origin xyz="0 0 0" rpy="1.57 0 1.57" />
   </xacro:imu_plugin_macro>
   <xacro:if value="$(arg enable_ground_truth)">
@@ -102,5 +102,5 @@
     >
       <inertia ixx="0.00001" ixy="0.0" ixz="0.0" iyy="0.00001" iyz="0.0" izz="0.00001" />
-      <origin xyz="0 0 0" rpy="-1.57 0 1.57" />
+      <origin xyz="0 0 0" rpy="1.57 0 1.57" />
     </xacro:imu_plugin_macro>
     <!-- Mount a generic odometry sensor providing ground truth. -->
